File: pcb/sotpotatis_pomodoro_timer/sotpotatis_pomodoro_timer.kicad_sch (KiCad schematic)
At the start: 23 parts, among them U1 ATtiny84A-P

Commit message: add: ADC input pin multiplexing added to PCB
Parts:
- added C2: 100n, Connector_PinSocket_2.54mm:PinSocket_1x02_P2.54mm_Vertical, symbol Device:C
- added R10, R7: 2.2k, Connector_PinSocket_2.54mm:PinSocket_1x02_P2.54mm_Vertical, symbol Device:R
- added R11: 5.1k, Connector_PinSocket_2.54mm:PinSocket_1x02_P2.54mm_Vertical, symbol Device:R
- added R8: 510, Connector_PinSocket_2.54mm:PinSocket_1x02_P2.54mm_Vertical, symbol Device:R
- added R9: 680, Connector_PinSocket_2.54mm:PinSocket_1x02_P2.54mm_Vertical, symbol Device:R
- added SW1: INCREASE_BTN, Button_Switch_THT:SW_PUSH-12mm, symbol Switch:SW_Push
- added SW2: PRESET_1_BTN, Button_Switch_THT:SW_PUSH-12mm, symbol Switch:SW_Push
- added SW3: PRESET_2_BTN, Button_Switch_THT:SW_PUSH-12mm, symbol Switch:SW_Push
- added SW4: PRESET_3_BTN, Button_Switch_THT:SW_PUSH-12mm, symbol Switch:SW_Push
- added SW5: DECREASE_BTN, Button_Switch_THT:SW_PUSH-12mm, symbol Switch:SW_Push
Connections:
- net GND: now also C2.2, SW1.2, SW2.2, SW3.2, SW4.2, SW5.2
- net PA0: now also C2.1, R7.2, R8.1, SW1.1; no longer R2.1
- net PA1: no longer R3.1
- net PA2: no longer R4.1
- net PA3: no longer R5.1
- net PA4: no longer R6.1
- net PA6: now also R6.1
- net VCC: now also R7.1
- net PB0: now reaches U1.2 (XTAL1/PB0)
- net PB0: now also R2.1
- net PB1: now reaches U1.3 (XTAL2/PB1)
- net PB1: now also R3.1
- net PB2: now reaches U1.5 (PB2)
- net PB2: now also R4.1
- net PA7: now reaches U1.6 (PA7)
- net PA7: now also R5.1
- new net: R10.1, R9.2, SW3.1
- new net: R10.2, R11.1, SW4.1
- new net: R11.2, SW5.1
- new net: R8.2, R9.1, SW2.1
Other:
- note added: "BTN_INPUT_MULTIPLEXING"
- note added: "LED_OUTPUT_CHARLIEPLEXING"
