File: pcb/sotpotatis_pomodoro_timer/sotpotatis_pomodoro_timer.kicad_sch (KiCad schematic)
At the start: 45 parts, among them J2 USB_C_PWR_IN, SW1 LEFT_BTN, SW2 PRESET_1_BTN, SW3 PRESET_2_BTN, SW4 PRESET_3_BTN, SW5 RIGHT_BTN, SW6 PWR_SWITCH, U1 ATtiny84A-P

Commit message: add: Backup spaghetti Charlieplexing wiring :)
Parts:
- added H1, H2, H3, H4: MountingHole, MountingHole:MountingHole_3.2mm_M3, symbol Mechanical:MountingHole
